File: PCB/RGB Controller/RGB Controller.sch (KiCad schematic (older format))
At the start: 58 parts, among them J1 Conn_01x06, J10 Conn_01x04, J11 Conn_01x03, J12 641737-1, J2 Conn_01x04, J3 Conn_01x04, J4 Conn_01x04, J5 Conn_01x04, J6 Conn_01x04, J7 Conn_01x04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

Commit message: Rev 0.1B hardware - Fixes Corsair Header pinout, 0.1A stencil compatible
Connections:
- net +5V: now also J11.3 (Pin_3); no longer J11.1 (Pin_1)
- net GND: now also J11.1 (Pin_1); no longer J11.3 (Pin_3)
Other:
- moved on the sheet: J11
Changed lines of the file:
@@
 	7400 5450 7600 5450
-Wire Wire Line
-	7750 5250 7600 5250
 Wire Wire Line
 	7500 5250 7500 5000
@@
 L Connector_Generic:Conn_01x03 J11
 U 1 1 5FC0450D
-P 7950 5250
-F 0 "J11" H 8030 5292 50  0000 L CNN
-F 1 "Conn_01x03" H 8030 5201 50  0000 L CNN
-F 2 "Custom Footprints:70555-0002" H 7950 5250 50  0001 C CNN
-F 3 "~" H 7950 5250 50  0001 C CNN
-F 4 "70555-0002" H 7950 5250 50  0001 C CNN "MPN"
-F 5 "WM4176-ND" H 7950 5250 50  0001 C CNN "Digi-Key_PN"
-	1    7950 5250
-	1    0    0    -1
+P 8350 5250
+F 0 "J11" H 8430 5292 50  0000 L CNN
+F 1 "Conn_01x03" H 8430 5201 50  0000 L CNN
+F 2 "Custom Footprints:70555-0002" H 8350 5250 50  0001 C CNN
+F 3 "~" H 8350 5250 50  0001 C CNN
+F 4 "70555-0002" H 8350 5250 50  0001 C CNN "MPN"
+F 5 "WM4176-ND" H 8350 5250 50  0001 C CNN "Digi-Key_PN"
+	1    8350 5250
+	-1   0    0    1
 $EndComp
 Connection ~ 7750 5150
@@
 	1    0    0    -1
 $EndComp
+Wire Wire Line
+	7750 5150 8550 5150
+Wire Wire Line
+	7600 5250 8550 5250
+Wire Wire Line
+	7750 5350 8550 5350
 $EndSCHEMATC
